Commit message: add friction

File: model/abstract/model.sdf.xacro (robot description, xacro)
@@ -128,4 +128,5 @@
 						<spring_stiffness>0</spring_stiffness>
 						<damping>0</damping>
+						<friction>0.0001</friction>
 					</dynamics>
 				</axis>
@@ -148,5 +149,9 @@
 		<xacro:body_omni_joint name="back_joint" child="omni_wheel_back_model::omni_wheel_rim_link"/>
 		<!--
-			<plugin name='omni_plugin' filename='/home/guir/gazebo/robot/mobile/wheel/3/omni/open_base/plugin/main/build/libmain.so'/>
+		<plugin name="omni_drive" filename="libgazebo_ros_omni_drive.so">
+			<joint>left_joint</joint>
+			<joint>right_joint</joint>
+			<joint>back_joint</joint>
+		</plugin>
 		-->
 	</model>

File: model/omni_wheel/model.sdf.xacro (robot description, xacro)
@@ -208,5 +208,5 @@
 						<spring_stiffness>0</spring_stiffness>
 						<damping>0</damping>
-						<friction>0</friction>
+						<friction>0.001</friction>
 					</dynamics>
 				</axis>
