Commit message: mitigate slipping problem

File: openbase_gazebo_models/models/simple_omni_wheel/model.sdf.xacro (robot description, xacro)
@@ -101,13 +101,13 @@
 				<xacro:insert_block name="pose"/>
 				<inertial>
-					<mass>0.00113845</mass>
+					<mass>0.00313845</mass>
 					<pose>0 0 0 0 0 0</pose>
 					<inertia>
-						<ixx>2.53776e-08</ixx>
+						<ixx>2.53776e-07</ixx>
 						<ixy>0</ixy>
 						<ixz>0</ixz>
-						<iyy>2.53776e-08</iyy>
+						<iyy>2.53776e-07</iyy>
 						<iyz>0</iyz>
-						<izz>1.47666e-08</izz>
+						<izz>1.47666e-07</izz>
 					</inertia>
 				</inertial>
@@ -209,5 +209,5 @@
 						<spring_stiffness>0</spring_stiffness>
 						<damping>0</damping>
-						<friction>0.002</friction>
+						<friction>0.001</friction>
 					</dynamics>
 				</axis>

Commit message: emit needless tags

File: openbase_gazebo_models/models/simple_omni_wheel/model.sdf.xacro (robot description, xacro)
@@ -1,21 +1,20 @@
-<?xml version='1.0'?>
-<sdf version='1.6' xmlns:xacro="http://www.ros.org/wiki/xacro">
-	<model name='simple_omni_wheel_model'>
+<?xml version="1.0"?>
+<sdf version="1.7" xmlns:xacro="http://www.ros.org/wiki/xacro">
+	<model name="simple_omni_wheel_model">
 		<xacro:macro name="omni_wheel_rim_link" params="name">
-			<link name='${name}'>
-				<pose>0 0 0 0 0 0</pose>
+			<link name="${name}">
 				<inertial>
+					<pose>0 0 0 0 ${pi/2} 0</pose>
 					<mass>0.00835758</mass>
 					<inertia>
-						<ixx>9.40333e-07</ixx>
+						<ixx>6.63684e-07</ixx>
 						<ixy>0</ixy>
 						<ixz>0</ixz>
 						<iyy>6.63684e-07</iyy>
 						<iyz>0</iyz>
-						<izz>6.63684e-07</izz>
+						<izz>9.40333e-07</izz>
 					</inertia>
-					<pose>0 -0.000343 0 0 0 0</pose>
 				</inertial>
-				<visual name='visual'>
+				<visual name="visual">
 					<pose>0 0 0 0 ${pi/2} 0</pose>
 					<geometry>
@@ -26,21 +25,11 @@
 					</geometry>
 					<material>
-						<lighting>true</lighting>
 						<script>
 							<uri>file://media/materials/scripts/gazebo.material</uri>
 							<name>Gazebo/Grey</name>
 						</script>
-						<ambient>0.3 0.3 0.3 1</ambient>
-						<diffuse>0.7 0.7 0.7 1</diffuse>
-						<specular>0.01 0.01 0.01 1</specular>
-						<emissive>0 0 0 1</emissive>
-						<shader type='vertex'>
-							<normal_map>__default__</normal_map>
-						</shader>
 					</material>
 				</visual>
-				<collision name='collision'>
-					<laser_retro>0</laser_retro>
-					<max_contacts>10</max_contacts>
+				<collision name="collision">
 					<pose>0 0 0 0 ${pi/2} 0</pose>
 					<geometry>
@@ -59,38 +48,5 @@
 								<slip2>0</slip2>
 							</ode>
-							<torsional>
-								<coefficient>1</coefficient>
-								<patch_radius>0</patch_radius>
-								<surface_radius>0</surface_radius>
-								<use_patch_radius>true</use_patch_radius>
-								<ode>
-									<slip>0</slip>
-								</ode>
-							</torsional>
 						</friction>
-						<bounce>
-							<restitution_coefficient>0</restitution_coefficient>
-							<threshold>1e+06</threshold>
-						</bounce>
-						<contact>
-							<collide_without_contact>false</collide_without_contact>
-							<collide_bitmask>1</collide_bitmask>
-							<ode>
-								<soft_cfm>0</soft_cfm>
-								<soft_erp>0.2</soft_erp>
-								<kp>1e+13</kp>
-								<kd>1</kd>
-								<max_vel>0.01</max_vel>
-								<min_depth>0</min_depth>
-							</ode>
-							<bullet>
-								<split_impulse>true</split_impulse>
-								<split_impulse_penetration_threshold>-0.01</split_impulse_penetration_threshold>
-								<soft_cfm>0</soft_cfm>
-								<soft_erp>0.2</soft_erp>
-								<kp>1e+13</kp>
-								<kd>1</kd>
-							</bullet>
-						</contact>
 					</surface>
 				</collision>
@@ -98,5 +54,5 @@
 		</xacro:macro>
 		<xacro:macro name="omni_wheel_roller_link" params="name *pose">
-			<link name='${name}'>
+			<link name="${name}">
 				<xacro:insert_block name="pose"/>
 				<inertial>
@@ -112,5 +68,5 @@
 					</inertia>
 				</inertial>
-				<visual name='visual'>
+				<visual name="visual">
 					<pose>0 0 0 0 0 0</pose>
 					<geometry>
@@ -121,21 +77,11 @@
 					</geometry>
 					<material>
-						<lighting>true</lighting>
 						<script>
 							<uri>file://media/materials/scripts/gazebo.material</uri>
-							<name>Gazebo/Grey</name>
+							<name>Gazebo/Black</name>
 						</script>
-						<ambient>0.03 0.03 0.03 1</ambient>
-						<diffuse>0.07 0.07 0.07 1</diffuse>
-						<specular>0.001 0.001 0.001 1</specular>
-						<emissive>0 0 0 1</emissive>
-						<shader type='vertex'>
-							<normal_map>__default__</normal_map>
-						</shader>
 					</material>
 				</visual>
-				<collision name='collision'>
-					<laser_retro>0</laser_retro>
-					<max_contacts>10</max_contacts>
+				<collision name="collision">
 					<pose>0 0 0 0 0 0</pose>
 					<geometry>
@@ -154,38 +100,5 @@
 								<slip2>0</slip2>
 							</ode>
-							<torsional>
-								<coefficient>1</coefficient>
-								<patch_radius>0</patch_radius>
-								<surface_radius>0</surface_radius>
-								<use_patch_radius>true</use_patch_radius>
-								<ode>
-									<slip>0</slip>
-								</ode>
-							</torsional>
 						</friction>
-						<bounce>
-							<restitution_coefficient>0</restitution_coefficient>
-							<threshold>1e+06</threshold>
-						</bounce>
-						<contact>
-							<collide_without_contact>false</collide_without_contact>
-							<collide_bitmask>1</collide_bitmask>
-							<ode>
-								<soft_cfm>0</soft_cfm>
-								<soft_erp>0.2</soft_erp>
-								<kp>1e+13</kp>
-								<kd>1</kd>
-								<max_vel>0.01</max_vel>
-								<min_depth>0</min_depth>
-							</ode>
-							<bullet>
-								<split_impulse>true</split_impulse>
-								<split_impulse_penetration_threshold>-0.01</split_impulse_penetration_threshold>
-								<soft_cfm>0</soft_cfm>
-								<soft_erp>0.2</soft_erp>
-								<kp>1e+13</kp>
-								<kd>1</kd>
-							</bullet>
-						</contact>
 					</surface>
 				</collision>
@@ -193,5 +106,5 @@
 		</xacro:macro>
 		<xacro:macro name="omni_wheel_joint" params="name child">
-			<joint name='${name}' type='revolute'>
+			<joint name="${name}" type="revolute">
 				<parent>omni_wheel_rim_link</parent>
 				<child>${child}</child>
@@ -199,10 +112,4 @@
 				<axis>
 					<xyz>0 0 1</xyz>
-					<limit>
-						<lower>-1.79769e+308</lower>
-						<upper>1.79769e+308</upper>
-						<effort>-1</effort>
-						<velocity>-1</velocity>
-					</limit>
 					<dynamics>
 						<spring_reference>0</spring_reference>
@@ -212,16 +119,4 @@
 					</dynamics>
 				</axis>
-				<physics>
-					<ode>
-						<limit>
-							<cfm>0</cfm>
-							<erp>0.2</erp>
-						</limit>
-						<suspension>
-							<cfm>0</cfm>
-							<erp>0.2</erp>
-						</suspension>
-					</ode>
-				</physics>
 			</joint>
 		</xacro:macro>
