Commit message: add camera, fix wheel configurations

File: openbase_gazebo_models/models/damped_omni4/model.sdf.xacro (robot description, xacro)
@@ -9,10 +9,10 @@
 				<pose>0 0 0 0 0 0</pose>
 				<inertia>
-					<ixx>0.00002035985530754</ixx>
+					<ixx>0.00018035985530754</ixx>
 					<ixy>0</ixy>
 					<ixz>0</ixz>
-					<iyy>0.00002035985530754</iyy>
+					<iyy>0.00018035985530754</iyy>
 					<iyz>0</iyz>
-					<izz>0.00003945961663220</izz>
+					<izz>0.00018945961663220</izz>
 				</inertia>
 			</inertial>
@@ -20,8 +20,7 @@
 				<pose>0 0 0 0 0 0</pose>
 				<geometry>
-					<cylinder>
-						<radius>0.030</radius>
-						<length>0.015</length>
-					</cylinder>
+					<box>
+						<size>0.14 0.14 0.015</size>
+					</box>
 				</geometry>
 				<material>
@@ -45,8 +44,7 @@
 				<pose>0 0 0 0 0 0</pose>
 				<geometry>
-					<cylinder>
-						<radius>0.030</radius>
-						<length>0.015</length>
-					</cylinder>
+					<box>
+						<size>0.14 0.14 0.015</size>
+					</box>
 				</geometry>
 				<surface>
@@ -99,20 +97,20 @@
 			<name>simple_omni_wheel_front_left_model</name>
 			<uri>model://simple_omni_wheel</uri>
-			<pose>${0.04*cos(pi*3/4)} ${0.04*sin(pi*3/4)} 0 0 0 ${pi*3/4}</pose>
+			<pose>${0.12*cos(pi*1/4)} ${0.12*sin(pi*1/4)} 0 0 0 ${pi*1/4}</pose>
+		</include>
+		<include>
+			<name>simple_omni_wheel_back_left_model</name>
+			<uri>model://simple_omni_wheel</uri>
+			<pose>${0.12*cos(pi*3/4)} ${0.12*sin(pi*3/4)} 0 0 0 ${pi*3/4}</pose>
+		</include>
+		<include>
+			<name>simple_omni_wheel_back_right_model</name>
+			<uri>model://simple_omni_wheel</uri>
+			<pose>${0.12*cos(pi*5/4)} ${0.12*sin(pi*5/4)} 0 0 0 ${pi*5/4}</pose>
 		</include>
 		<include>
 			<name>simple_omni_wheel_front_right_model</name>
 			<uri>model://simple_omni_wheel</uri>
-			<pose>${0.04*cos(pi*1/4)} ${0.04*sin(pi*1/4)} 0 0 0 ${pi*1/4}</pose>
-		</include>
-		<include>
-			<name>simple_omni_wheel_back_left_model</name>
-			<uri>model://simple_omni_wheel</uri>
-			<pose>${0.04*cos(pi*5/4)} ${0.04*sin(pi*5/4)} 0 0 0 ${pi*5/4}</pose>
-		</include>
-		<include>
-			<name>simple_omni_wheel_back_right_model</name>
-			<uri>model://simple_omni_wheel</uri>
-			<pose>${0.04*cos(pi*7/4)} ${0.04*sin(pi*7/4)} 0 0 0 ${pi*7/4}</pose>
+			<pose>${0.12*cos(pi*7/4)} ${0.12*sin(pi*7/4)} 0 0 0 ${pi*7/4}</pose>
 		</include>
 		<xacro:macro name="body_omni_conn" params="prefix omni_link">

File: openbase_gazebo_models/models/nav_omni4/model.sdf.xacro (robot description, xacro)
@@ -8,5 +8,5 @@
 		</include>
 		<link name="lidar_link">
-			<pose>0 0 0.035 0 0 0</pose>
+			<pose>0 0 0.05 0 0 0</pose>
 			<inertial>
 				<mass>0.001</mass>
@@ -53,8 +53,67 @@
 			</sensor>
 		</link>
+		<link name="camera_link">
+			<pose>0.07 0 0.05 0 0 0</pose>
+			<inertial>
+				<mass>0.001</mass>
+				<inertia>
+					<ixx>0.00001</ixx>
+					<ixy>0</ixy>
+					<ixz>0</ixz>
+					<iyy>0.00001</iyy>
+					<iyz>0</iyz>
+					<izz>0.00001</izz>
+				</inertia>
+			</inertial>
+			<visual name="visual">
+				<geometry>
+					<box>
+						<size>0.01 0.015 0.01</size>
+					</box>
+				</geometry>
+			</visual>
+			<sensor name="camera1" type="camera">
+				<update_rate>20.0</update_rate>
+				<camera name="head">
+					<horizontal_fov>1.3962634</horizontal_fov>
+					<image>
+						<width>800</width>
+						<height>800</height>
+						<format>R8G8B8</format>
+					</image>
+					<clip>
+						<near>0.02</near>
+						<far>300</far>
+					</clip>
+					<noise>
+						<type>gaussian</type>
+						<mean>0.0</mean>
+						<stddev>0.007</stddev>
+					</noise>
+				</camera>
+				<plugin name="camera_controller" filename="libgazebo_ros_camera.so">
+					<alwaysOn>true</alwaysOn>
+					<updateRate>0.0</updateRate>
+					<cameraName>nav_omni4/camera1</cameraName>
+					<imageTopicName>image_raw</imageTopicName>
+					<cameraInfoTopicName>camera_info</cameraInfoTopicName>
+					<frameName>camera_link</frameName>
+					<hackBaseline>0.07</hackBaseline>
+					<distortionK1>0.0</distortionK1>
+					<distortionK2>0.0</distortionK2>
+					<distortionK3>0.0</distortionK3>
+					<distortionT1>0.0</distortionT1>
+					<distortionT2>0.0</distortionT2>
+				</plugin>
+			</sensor>
+		</link>
 		<joint name="lidar_joint" type="fixed">
 			<parent>damped_omni4_model::body_link</parent>
 			<child>lidar_link</child>
 		</joint>
+		<joint name="camera_joint" type="fixed">
+			<parent>damped_omni4_model::body_link</parent>
+			<child>camera_link</child>
+		</joint>
 	</model>
 </sdf>

File: openbase_gazebo_models/models/simple_omni_wheel/model.sdf.xacro (robot description, xacro)
@@ -209,5 +209,5 @@
 						<spring_stiffness>0</spring_stiffness>
 						<damping>0</damping>
-						<friction>0.001</friction>
+						<friction>0.002</friction>
 					</dynamics>
 				</axis>

Commit message: first nav2 demo

File: openbase_gazebo_models/models/damped_omni4/model.sdf.xacro (robot description, xacro)
@@ -187,5 +187,5 @@
 			<joint>back_left_rotational_joint</joint>
 			<joint>back_right_rotational_joint</joint>
-			<wheel_radius>0.05</wheel_radius>
+			<wheel_radius>0.018</wheel_radius>
 		</plugin>
 	</model>

File: openbase_gazebo_models/models/nav_omni4/model.sdf.xacro (robot description, xacro)
@@ -144,4 +144,38 @@
 			</sensor>
 		</link>
+		<link name="dummy_link_1">
+			<inertial>
+				<mass>0.001</mass>
+				<inertia>
+					<ixx>0.00001</ixx>
+					<ixy>0</ixy>
+					<ixz>0</ixz>
+					<iyy>0.00001</iyy>
+					<iyz>0</iyz>
+					<izz>0.00001</izz>
+				</inertia>
+			</inertial>
+		</link>
+		<link name="dummy_link_2">
+			<inertial>
+				<mass>0.001</mass>
+				<inertia>
+					<ixx>0.00001</ixx>
+					<ixy>0</ixy>
+					<ixz>0</ixz>
+					<iyy>0.00001</iyy>
+					<iyz>0</iyz>
+					<izz>0.00001</izz>
+				</inertia>
+			</inertial>
+		</link>
+		<joint name="dummy_joint1" type="revolute">
+			<parent>damped_omni4_model::body_link</parent>
+			<child>dummy_link_1</child>
+		</joint>
+		<joint name="dummy_joint2" type="revolute">
+			<parent>damped_omni4_model::body_link</parent>
+			<child>dummy_link_2</child>
+		</joint>
 		<joint name="lidar_joint" type="fixed">
 			<parent>damped_omni4_model::body_link</parent>
@@ -152,8 +186,31 @@
 			<child>camera_link</child>
 		</joint>
+		<!--
 		<plugin name="wheel_odometry" filename="libgazebo_ros_wheel_odometry.so">
 			<publish_odom_msg>true</publish_odom_msg>
 			<publish_tf>true</publish_tf>
+			<robot_base_frame>base_link</robot_base_frame>
 		</plugin>
+		-->
+      <plugin name="turtlebot3_diff_drive" filename="libgazebo_ros_diff_drive.so">
+        <update_rate>30</update_rate>
+        <!-- wheels -->
+        <left_joint>dummy_joint1</left_joint>
+        <right_joint>dummy_joint2</right_joint>
+        <!-- kinematics -->
+        <wheel_separation>0.287</wheel_separation>
+        <wheel_diameter>0.066</wheel_diameter>
+        <!-- limits -->
+        <max_wheel_torque>0</max_wheel_torque>
+        <max_wheel_acceleration>0.0</max_wheel_acceleration>
+        <command_topic>cmd_vel</command_topic>
+        <!-- output -->
+        <publish_odom>true</publish_odom>
+        <publish_odom_tf>true</publish_odom_tf>
+        <publish_wheel_tf>false</publish_wheel_tf>
+        <odometry_topic>odom</odometry_topic>
+        <odometry_frame>odom</odometry_frame>
+        <robot_base_frame>base_link</robot_base_frame>
+      </plugin>
 	</model>
 </sdf>

Commit message: fixed formulae for computing wheel velocities

File: openbase_gazebo_models/models/damped_omni4/model.sdf.xacro (robot description, xacro)
@@ -187,5 +187,5 @@
 			<joint>back_left_rotational_joint</joint>
 			<joint>back_right_rotational_joint</joint>
-			<wheel_radius>0.018</wheel_radius>
+			<wheel_radius>0.0229</wheel_radius>
 		</plugin>
 	</model>

File: openbase_gazebo_models/models/nav_omni4/model.sdf.xacro (robot description, xacro)
@@ -111,5 +111,5 @@
 			<sensor name="depth_camera" type="depth">
 				<visualize>true</visualize>
-				<update_rate>30.0</update_rate>
+				<update_rate>1.0</update_rate>
 				<camera name="camera">
 					<horizontal_fov>1.047198</horizontal_fov>
@@ -187,11 +187,16 @@
 		</joint>
 		<plugin name="wheel_odometry" filename="libgazebo_ros_wheel_odometry.so">
+			<update_rate>30.0</update_rate>
 			<publish_odom_msg>true</publish_odom_msg>
 			<publish_tf>true</publish_tf>
 			<robot_base_frame>base_link</robot_base_frame>
+			<joint>damped_omni4_model::front_left_rotational_joint</joint>
+			<joint>damped_omni4_model::back_left_rotational_joint</joint>
+			<joint>damped_omni4_model::back_right_rotational_joint</joint>
+			<joint>damped_omni4_model::front_right_rotational_joint</joint>
 		</plugin>
-	  <!--
+		<!--
       <plugin name="turtlebot3_diff_drive" filename="libgazebo_ros_diff_drive.so">
-        <update_rate>30</update_rate>
+        <update_rate>30.0</update_rate>
         <left_joint>dummy_joint1</left_joint>
         <right_joint>dummy_joint2</right_joint>
@@ -202,5 +207,5 @@
         <command_topic>cmd_vel</command_topic>
         <publish_odom>true</publish_odom>
-        <publish_odom_tf>true</publish_odom_tf>
+        <publish_odom_tf>false</publish_odom_tf>
         <publish_wheel_tf>false</publish_wheel_tf>
         <odometry_topic>odom</odometry_topic>

File: openbase_gazebo_models/models/omni4/model.sdf.xacro (robot description, xacro)
@@ -37,20 +37,20 @@
 			<name>simple_omni_wheel_front_left_model</name>
 			<uri>model://primitive_omni_wheel</uri>
-			<pose>${box_r*cos(pi*1/4)} ${box_r*sin(pi*1/4)} 0 0 0 ${pi*3/4}</pose>
+			<pose>${box_r*cos(pi*1/4)} ${box_r*sin(pi*1/4)} 0 0 0 ${-pi*1/4}</pose>
 		</include>
 		<include>
 			<name>simple_omni_wheel_back_left_model</name>
 			<uri>model://primitive_omni_wheel</uri>
-			<pose>${box_r*cos(pi*3/4)} ${box_r*sin(pi*3/4)} 0 0 0 ${pi*5/4}</pose>
+			<pose>${box_r*cos(pi*3/4)} ${box_r*sin(pi*3/4)} 0 0 0 ${pi*1/4}</pose>
 		</include>
 		<include>
 			<name>simple_omni_wheel_back_right_model</name>
 			<uri>model://primitive_omni_wheel</uri>
-			<pose>${box_r*cos(pi*5/4)} ${box_r*sin(pi*5/4)} 0 0 0 ${pi*7/4}</pose>
+			<pose>${box_r*cos(pi*5/4)} ${box_r*sin(pi*5/4)} 0 0 0 ${pi*3/4}</pose>
 		</include>
 		<include>
 			<name>simple_omni_wheel_front_right_model</name>
 			<uri>model://primitive_omni_wheel</uri>
-			<pose>${box_r*cos(pi*7/4)} ${box_r*sin(pi*7/4)} 0 0 0 ${pi*1/4}</pose>
+			<pose>${box_r*cos(pi*7/4)} ${box_r*sin(pi*7/4)} 0 0 0 ${-pi*3/4}</pose>
 		</include>
 		<xacro:macro name="body_omni_conn" params="prefix omni_link">
@@ -125,5 +125,15 @@
 			<joint>back_left_rotational_joint</joint>
 			<joint>back_right_rotational_joint</joint>
-			<wheel_radius>0.06</wheel_radius>
+			<wheel_radius>0.063</wheel_radius>
+		</plugin>
+		<plugin name="wheel_odometry" filename="libgazebo_ros_wheel_odometry.so">
+			<update_rate>30.0</update_rate>
+			<publish_odom_msg>true</publish_odom_msg>
+			<publish_tf>true</publish_tf>
+			<robot_base_frame>base_link</robot_base_frame>
+			<joint>front_left_rotational_joint</joint>
+			<joint>back_left_rotational_joint</joint>
+			<joint>back_right_rotational_joint</joint>
+			<joint>front_right_rotational_joint</joint>
 		</plugin>
 	</model>

File: openbase_gazebo_models/models/primitive_omni_wheel/model.sdf.xacro (robot description, xacro)
@@ -12,4 +12,5 @@
 		)) }"/>
 	-->
+	<!--
 	<xacro:property name="omni_wheel_params" value="${
 		xacro.dotify(dict(
@@ -20,4 +21,5 @@
 			num_rollers=4
 		)) }"/>
+	-->
 	<!--
 	<xacro:property name="omni_wheel_params" value="${
@@ -30,5 +32,4 @@
 		)) }"/>
 	-->
-	<!--
 	<xacro:property name="omni_wheel_params" value="${
 		xacro.dotify(dict(
@@ -39,5 +40,4 @@
 			num_rollers=16
 		)) }"/>
-	-->
 	<xacro:omni_wheel_model name="primitive_omni_wheel_model" params="${
 		xacro.dotify(
