Commit message: add top_level_tags

File: openbase_gazebo_models/models/omni4/model.sdf.xacro (robot description, xacro)
@@ -55,5 +55,4 @@
 		</include>
 		<xacro:macro name="body_omni_conn" params="prefix omni_link">
-				<!--
 			<joint name='${prefix}_linear_joint' type='fixed'>
 				<parent>body_link</parent>
@@ -79,19 +78,18 @@
 			<link name='${prefix}_wheel_base_link'>
 				<inertial>
-					<mass>0.001</mass>
+					<mass>0.1</mass>
 					<inertia>
-						<ixx>0.00001</ixx>
+						<ixx>0.0002</ixx>
 						<ixy>0</ixy>
 						<ixz>0</ixz>
-						<iyy>0.00001</iyy>
+						<iyy>0.0002</iyy>
 						<iyz>0</iyz>
-						<izz>0.00001</izz>
+						<izz>0.0002</izz>
 					</inertia>
 				</inertial>
 			</link>
-				-->
 			<joint name='${prefix}_rotational_joint' type='revolute'>
-				<!--<parent>${prefix}_wheel_base_link</parent>-->
-				<parent>body_link</parent>
+				<parent>${prefix}_wheel_base_link</parent>
+				<!--<parent>body_link</parent>-->
 				<child>${omni_link}</child>
 				<axis>

File: openbase_gazebo_models/models/primitive_omni_wheel/model.sdf.xacro (robot description, xacro)
@@ -14,4 +14,13 @@
 	<xacro:property name="omni_wheel_params" value="${
 		xacro.dotify(dict(
+			rim_radius=0.06, rim_length=0.029,
+			roller_radius=0.012, roller_length=0.030,
+			rim_inner_radius=0.050, rim_inner_length=0.008,
+			rim_mass=0.30, roller_mass=0.03,
+			num_rollers=4
+		)) }"/>
+	<!--
+	<xacro:property name="omni_wheel_params" value="${
+		xacro.dotify(dict(
 			rim_radius=0.06, rim_length=0.025,
 			roller_radius=0.008, roller_length=0.020,
@@ -20,12 +29,13 @@
 			num_rollers=8
 		)) }"/>
+	-->
 	<!--
 	<xacro:property name="omni_wheel_params" value="${
 		xacro.dotify(dict(
-			rim_radius=0.06, rim_length=0.029,
-			roller_radius=0.012, roller_length=0.030,
-			rim_inner_radius=0.050, rim_inner_length=0.008,
-			rim_mass=0.30, roller_mass=0.03,
-			num_rollers=4
+			rim_radius=0.06, rim_length=0.025,
+			roller_radius=0.008, roller_length=0.010,
+			rim_inner_radius=0.055, rim_inner_length=0.008,
+			rim_mass=0.30, roller_mass=0.01,
+			num_rollers=16
 		)) }"/>
 	-->
@@ -44,4 +54,8 @@
 					omni_wheel_params.roller_length
 				)
-			)) }"/>
+			)) }">
+		<top_level_tags>
+			<pose>0 0 0.1 0 0 0</pose>
+		</top_level_tags>
+	</xacro:omni_wheel_model>
 </sdf>

File: openbase_gazebo_models/models/primitive_omni_wheel/parts.sdf.xacro (robot description, xacro)
@@ -156,6 +156,7 @@
 		</xacro:unless>
 	</xacro:macro>
-	<xacro:macro name="omni_wheel_model" params="name params">
+	<xacro:macro name="omni_wheel_model" params="name params **top_level_tags">
 		<model name="${name}">
+			<xacro:insert_block name="top_level_tags"/>
 			<xacro:omni_wheel_rim_link name="rim_link" radius="${params.rim_radius}" length="${params.rim_length}" mass="${params.rim_mass}" inertia="${params.rim_inertia}"/>
 			<xacro:omni_wheel_model_rollers i="0" params="${params}"/>

File: openbase_gazebo_models/models/unicycle_wheel_2/model.sdf.xacro (robot description, xacro)
@@ -1,6 +1,6 @@
-<?xml version='1.0'?>
-<sdf version='1.6' xmlns:xacro="http://www.ros.org/wiki/xacro">
-	<model name='unicycle_wheel_model'>
-		<pose>0 0 0.01 0 0 0</pose>
+<?xml version="1.0"?>
+<sdf version="1.6" xmlns:xacro="http://www.ros.org/wiki/xacro">
+	<model name="unicycle_wheel_2_model">
+		<pose>0 0 0.02 0 0 0</pose>
 		<link name='unicycle_wheel_rim_link'>
 			<pose>0 0 0.005 0 0 0</pose>
@@ -173,5 +173,5 @@
 		</joint>
 		<link name="unicycle_wheel_base_link">
-			<kinematic>false</kinematic>
+			<kinematic>true</kinematic>
 			<inertial>
 				<mass>0.001</mass>
@@ -185,5 +185,4 @@
 				</inertia>
 			</inertial>
-			<!--
 			<visual name="visual">
 				<geometry>
@@ -193,7 +192,5 @@
 				</geometry>
 			</visual>
-			-->
 		</link>
-		<!--
 		<plugin name="indep_steer_drive" filename="libgazebo_ros_indep_steer_drive.so">
 			<unicycle_joints>
@@ -203,5 +200,4 @@
 			<wheel_radius>0.05</wheel_radius>
 		</plugin>
-		-->
 	</model>
 </sdf>

Commit message: add translation matrix

File: openbase_gazebo_models/models/omni4/model.sdf.xacro (robot description, xacro)
@@ -7,4 +7,5 @@
 		<xacro:property name="box_inertia" value="${xacro.dotify(cuboid_inertia(box_mass, box_geom.wx, box_geom.wy, box_geom.wz))}"/>
 		<xacro:property name="box_r" value="${hypot(box_geom.wx/2, box_geom.wy/2)}"/>
+		<xacro:property name="wheel_r" value="0.063"/>
 		<pose>0 0 0.2 0 0 0</pose>
 		<link name='body_link'>
@@ -125,5 +126,5 @@
 			<joint>back_left_rotational_joint</joint>
 			<joint>back_right_rotational_joint</joint>
-			<wheel_radius>0.063</wheel_radius>
+			<wheel_radius>${wheel_r}</wheel_radius>
 		</plugin>
 		<plugin name="wheel_odometry" filename="libgazebo_ros_wheel_odometry.so">
@@ -136,4 +137,7 @@
 			<joint>back_right_rotational_joint</joint>
 			<joint>front_right_rotational_joint</joint>
+			<row>${-wheel_r/(2*sqrt(2))} ${-wheel_r/(2*sqrt(2))} ${wheel_r/(2*sqrt(2))} ${wheel_r/(2*sqrt(2))}</row>
+			<row>${wheel_r/(2*sqrt(2))} ${-wheel_r/(2*sqrt(2))} ${-wheel_r/(2*sqrt(2))} ${wheel_r/(2*sqrt(2))}</row>
+			<row>${wheel_r/(4*box_r)} ${wheel_r/(4*box_r)} ${wheel_r/(4*box_r)} ${wheel_r/(4*box_r)}</row>
 		</plugin>
 	</model>
